File: micromouse_pcb/micromouse_pcb.kicad_pcb (KiCad board)
At the start: 2 copper layers, 112.6 x 141.7 mm, 58 parts, among them J101 Conn_01x03, J102 Conn_01x06, J103 Conn_02x20_Odd_Even, J104 Conn_01x02, J105 Conn_01x06, J106 Conn_01x02, J111 Conn_01x06, Q101 BS170, Q102 SFH313FA, Q103 SFH313FA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

Commit message: first iteration of pin assignments and routing done
Parts:
- removed H102: MountingHole_Pad, MountingHole:MountingHole_2.2mm_M2_DIN965_Pad
- removed U101: Teensy4.1, MCU_TEENSY_Footprint:MODULE_DEV-16771
- added C109: 0.1 uF, Capacitor_SMD:C_0805_2012Metric, B.Cu at (145.7, 110.1)
- added C110: 4.7uF, Capacitor_SMD:C_0805_2012Metric, B.Cu at (142.7, 110.1)
- added C111: 4.7uF, Capacitor_SMD:C_0805_2012Metric, B.Cu at (132.9, 132.2)
- added C112: 10uF, Capacitor_SMD:C_0805_2012Metric, B.Cu at (132.9, 134.4)
- added U104: Teensy4.1_bare, MCU_TEENSY_Footprint:Teensy41_bare_pins, F.Cu at (83.3, 120.8)
- added U105: MCP3004, Package_DIP:DIP-14_W7.62mm, F.Cu at (97.8, 152.8)
- J103: value Conn_02x20_Odd_Even -> Conn_01x10; footprint Connector_PinHeader_2.54mm:PinHeader_2x20_P2.54mm_Vertical -> Connector_PinHeader_2.54mm:PinHeader_1x10_P2.54mm_Vertical
- U103: value ~ -> L293D; footprint Regulator_Pololu_D24V22FX:D24V22FX -> Package_DIP:DIP-16_W7.62mm
- moved H103 164.8 mm to (2.17, 2.17), turned to 0 degrees
- moved H110 101.8 mm to (263.4, 128.9)
- moved H111 101.8 mm to (263.4, 92.0)
- moved H109 101.8 mm to (226.4, 128.9)
- moved H112 101.8 mm to (226.4, 92.0)
- moved J101 91.2 mm to (230.6, 138.9)
- moved J102 91.2 mm to (240.2, 138.8)
- moved U103 76.8 mm to (131.8, 111.7), turned to 0 degrees
- moved J103 43.1 mm to (95.3, 135.7)
- moved J111 17.8 mm to (111.7, 89.3)
- moved J104 11.3 mm to (151.1, 38.0), turned to 90 degrees
- moved C104 7.48 mm to (83.9, 159.5)
- moved D102 7.48 mm to (78.2, 162.9)
- moved R110 7.48 mm to (83.2, 162.4)
- moved Q103 7.48 mm to (87.9, 162.7)
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Connections:
- J103 pad 1: unconnected-(J103-Pin_1-Pad1) -> /IR_EMITTER_1
- J103 pad 10: unconnected-(J103-Pin_10-Pad10) -> /IR_EMITTER_4
- J103 pad 2: unconnected-(J103-Pin_2-Pad2) -> /IR_EMITTER_2
- J103 pad 3: unconnected-(J103-Pin_3-Pad3) -> /RPI_3V3
- J103 pad 4: unconnected-(J103-Pin_4-Pad4) -> GND
- J103 pad 5: unconnected-(J103-Pin_5-Pad5) -> /RPI_CLK
- J103 pad 6: unconnected-(J103-Pin_6-Pad6) -> /RPI_MISO
- J103 pad 7: unconnected-(J103-Pin_7-Pad7) -> /RPI_MOSI
- J103 pad 8: unconnected-(J103-Pin_8-Pad8) -> /RPI_CS
- J103 pad 9: unconnected-(J103-Pin_9-Pad9) -> /IR_EMITTER_3
- J105 pad 2: /MOTOR1_OUTB -> /ML_OUTB
- J105 pad 3: /MOTOR1_OUTA -> /ML_OUTA
- J105 pad 4: /5V_REGULATED -> /3V3_REGULATED
- J105 pad 5: /MOTOR1_M1 -> /ML_2
- J105 pad 6: /MOTOR1_M2 -> /ML_1
- J111 pad 2: /MOTOR2_OUTB -> /MR_OUTB
- J111 pad 3: /MOTOR2_OUTA -> /MR_OUTA
- J111 pad 4: /5V_REGULATED -> /3V3_REGULATED
- J111 pad 5: /MOTOR2_M1 -> /MR_2
- J111 pad 6: /MOTOR2_M2 -> /MR_1
- U102 pad 3: /RPI_5V -> /VBAT
- U103 pad 1: unconnected-(U103-PG-Pad1) -> /3V3_REGULATED
- U103 pad 2: unconnected-(U103-EN-Pad2) -> /ML_IN_2
- U103 pad 3: /VBAT -> /ML_2
- U103 pad 4: GND -> /MGND
- U103 pad 5: /5V_REGULATED -> /MGND
- U103 pad 6: GND -> /ML_1
Routing:
- net /3V3_REGULATED: track 0.00 -> 315.5 mm, vias 0 -> 8
- net /VBAT: track 0.00 -> 175.7 mm, vias 0 -> 4
- net /MR_2: track 0.00 -> 58.5 mm, vias 0 -> 2
- net /ML_IN_2: track 0.00 -> 53.3 mm, vias 0 -> 1
- net /MR_IN_1: track 0.00 -> 47.8 mm, vias 0 -> 1
- net /ML_1: track 0.00 -> 47.8 mm, vias 0 -> 2
- net /IR_RECEIVER_3: track 0.00 -> 45.3 mm, vias 0 -> 1
- net /MR_1: track 0.00 -> 45.0 mm, vias 0 -> 2
- net /IR_RECEIVER_1: track 0.00 -> 44.3 mm, vias 0 -> 1
- net /ML_2: track 0.00 -> 42.2 mm, vias 0 -> 2
- net /MR_IN_2: track 0.00 -> 40.4 mm, vias 0 -> 1
- net /ML_IN_1: track 0.00 -> 39.3 mm, vias 0 -> 1
- net /IR_EMITTER_4: track 0.00 -> 32.1 mm, vias 0 -> 2
- net /IR_EMITTER_2: track 0.00 -> 31.8 mm, vias 0 -> 2
- net /IR_EMITTER_1: track 0.00 -> 27.1 mm, vias 0 -> 1
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- added copper zone on B.Cu, net /MGND
- added copper zone on F.Cu, net GND
Other:
- board size 112.6 x 141.7 mm -> 106.5 x 143.3 mm
- board text added: "GND"
- board text added: "GPIO"
- board text added: "Left Motor"
- board text added: "RPI_3V3"
- board text added: "RPI_CLK"
- board text added: "RPI_CS"
- board text added: "RPI_MISO"
- board text added: "RPI_MOSI"
- board text added: "Right Motor"
- board text added: "USB"
- board text removed: "Motor 1"
- board text removed: "Motor 2"

Commit message: cleaned up schematic
Parts:
- removed H103: MountingHole_Pad, MountingHole:MountingHole_2.2mm_M2_DIN965_Pad
- removed H109, H110, H111, H112: MountingHole_Pad, MountingHole:MountingHole_3.2mm_M3_DIN965_Pad
- removed J101: Conn_01x03, Connector_PinHeader_2.54mm:PinHeader_1x03_P2.54mm_Vertical
- removed J102: Conn_01x06, Connector_PinHeader_2.54mm:PinHeader_1x06_P2.54mm_Vertical
Other:
- board text removed: "L298N Motor Driver"

Commit message: updated pcb
Parts:
- removed H101: MountingHole_Pad, MountingHole:MountingHole_2.2mm_M2_DIN965_Pad
- added H103: MountingHole_Pad, MountingHole:MountingHole_2.2mm_M2_DIN965_Pad, F.Cu at (156.6, 58.2)
- added J102: Conn_02x02_Counter_Clockwise, Connector_PinHeader_2.54mm:PinHeader_2x02_P2.54mm_Vertical, F.Cu at (105.8, 92.3)
- added J108: Conn_01x04, Connector_PinHeader_2.54mm:PinHeader_1x04_P2.54mm_Vertical, F.Cu at (156.2, 123.1)
- added SW101: SW_SPST, Connector_PinHeader_2.54mm:PinHeader_1x02_P2.54mm_Vertical, F.Cu at (151.2, 46.4)
- C109, C110: moved to F.Cu
- R103: value 50 Ohm -> 51Ohm
- R110, R113: value 50 Ohm -> 51 Ohm
- moved J111 3.04 mm to (112.1, 92.3)
- moved J105 2.91 mm to (102.0, 92.3)
- moved U105 1.46 mm to (98.2, 151.4)
- moved C109 1.05 mm to (144.8, 110.7)
- moved C110 0.73 mm to (142.2, 110.7)
- moved H108 0.13 mm to (114.4, 75.5)
- moved H105 0.13 mm to (56.4, 75.5)
- moved H106 0.12 mm to (114.4, 26.4)
- moved H107 0.12 mm to (56.4, 26.4)
- moved U102 0.05 mm to (160.5, 61.5)
Connections:
- J104 pad 1: /VBAT -> Net-(J104-Pin_1)
- U104 pad 15: /TEENSY_3V3 -> unconnected-(U104-3V3-Pad15)
- U104 pad 46: /TEENSY_3V3 -> unconnected-(U104-3V3-Pad46)
Routing:
- net /IR_RECEIVER_4: track 6.81 -> 67.4 mm, vias 1 -> 3
- net GND: track 18.3 -> 0.00 mm, vias 1 -> 0
- net /MR_1: track 45.0 -> 55.9 mm
- net /3V3_REGULATED: track 315.5 -> 324.7 mm, vias 8 -> 7
- net Net-(J104-Pin_1): track 0.00 -> 8.35 mm
- net /MR_2: track 58.5 -> 66.8 mm
- net /IR_EMITTER_2: track 31.8 -> 36.3 mm
- net /RPI_3V3: track 9.55 -> 13.2 mm
- net /MR_OUTA: track 20.6 -> 23.3 mm
- net /IR_EMITTER_4: track 32.1 -> 34.4 mm
- net /MR_OUTB: track 24.2 -> 26.2 mm
- net /ML_OUTB: track 23.3 -> 25.1 mm
- net /ML_OUTA: track 20.2 -> 21.6 mm
- net /VBAT: track 175.7 -> 174.4 mm, vias 4 -> 2
- net /RPI_MOSI: track 9.55 -> 8.26 mm
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Other:
- outline, holes or cut-outs redrawn
- board text added: "3V3_R"
- board text added: "Adam Casselman Arna Bharadwaj Siddhant Panse"
- board text added: "MGND"
- board text added: "ML_OUTA"
- board text added: "ML_OUTB"
- board text added: "MR_OUTA"
- board text added: "MR_OUTB"
- board text added: "VBAT"
- board text removed: "Left Motor"
- board text removed: "Right Motor"

Commit message: added mounting holes
Parts:
- moved J106 26.9 mm to (143.3, 56.4)
- moved H103 22.8 mm to (143.4, 76.8)
- moved J104 18.4 mm to (150.1, 56.4)
- moved H104 15.2 mm to (156.6, 63.6)
- moved SW101 9.18 mm to (156.6, 53.8)
- moved U102 5.40 mm to (160.5, 66.9)
Routing:
- net /IR_EMITTER_4: track 34.4 -> 29.9 mm, vias 2 -> 1
- net /IR_RECEIVER_1: track 45.4 -> 41.0 mm
- net /VBAT: track 174.4 -> 171.3 mm
- net /3V3_REGULATED: track 324.7 -> 322.5 mm
- net Net-(J104-Pin_2): track 5.39 -> 7.55 mm
- net Net-(J104-Pin_1): track 8.35 -> 7.59 mm
- net /IR_EMITTER_3: track 19.9 -> 20.6 mm
- net /IR_RECEIVER_4: track 67.4 -> 66.8 mm
Other:
- outline, holes or cut-outs redrawn
- board text added: "Adam Casselman Arna Bhardwaj Siddhant Panse 2025"
- board text added: "Shift regulators and connectors down"
- board text removed: "Adam Casselman Arna Bharadwaj Siddhant Panse"
