File: micromouse_pcb/micromouse_pcb.kicad_sch (KiCad schematic)
At the start: 7 parts, among them J101 Conn_01x03, J102 Conn_01x06, J103 Conn_02x20_Odd_Even, J104 Conn_01x02, J105 Conn_01x02, J106 Conn_01x02, U101 Teensy4.1

Commit message: added regulators and motor encoders schematic
Parts:
- removed J105: Conn_01x02, Connector_JST:JST_PH_B2B-PH-K_1x02_P2.00mm_Vertical, symbol Connector_Generic:Conn_01x02
- added C101, C103, C105, C107: 4.7 uF, Capacitor_SMD:C_0805_2012Metric, symbol Device:C
- added C102, C104, C106, C108: 0.1 uF, Capacitor_SMD:C_0805_2012Metric, symbol Device:C
- added D101, D102, D103, D104: INL-5AMIR15, LED_THT:LED_D3.0mm_IRBlack, symbol LED:IR204A
- added J105, J111: Conn_01x06, Connector_PinHeader_2.54mm:PinHeader_1x06_P2.54mm_Vertical, symbol Connector_Generic:Conn_01x06
- added J107, J109: Conn_01x05, Connector_PinHeader_2.54mm:PinHeader_1x05_P2.54mm_Vertical, symbol Connector_Generic:Conn_01x05
- added J108, J110: Conn_01x01, Connector_PinHeader_2.54mm:PinHeader_1x01_P2.54mm_Vertical, symbol Connector_Generic:Conn_01x01
- added Q101, Q106, Q107, Q108: BS170, Package_TO_SOT_THT:TO-92_Inline, symbol Transistor_FET:BS170
- added Q102, Q103, Q104, Q105: SFH313FA, LED_THT:LED_D5.0mm_Clear, symbol Sensor_Optical:SFH300
- added R101, R108, R111, R114: 100, Resistor_SMD:R_0805_2012Metric, symbol Device:R_US
- added R102, R109, R112, R115: 47K, Resistor_SMD:R_0805_2012Metric, symbol Device:R_US
- added R103, R110, R113, R116: 50 Ohm, Resistor_SMD:R_0805_2012Metric, symbol Device:R_US
- added R104, R105, R106, R107: 1.8k, Resistor_SMD:R_0805_2012Metric, symbol Device:R_US
Connections:
- net VIN is gone; now on net VBAT: J101.3 (Pin_3)
- net GND: now also C101.2, C102.2, C103.2, C104.2, C105.2, C106.2, C107.2, C108.2, J105.1 (Pin_1), J107.4 (Pin_4), J108.1 (Pin_1), J109.4 (Pin_4), J110.1 (Pin_1), J111.1 (Pin_1), Q101.3 (S), Q106.3 (S), Q107.3 (S), Q108.3 (S), R102.2, R104.2, R105.2, R106.2, R107.2, R109.2, R112.2, R115.2
- net VBAT: now also J109.3 (Pin_3)
- net at J104.2 (Pin_2): now also J106.1 (Pin_1)
- net 5V_REGULATED: now reaches U101.48 (VIN)
- net 5V_REGULATED: now also J105.4 (Pin_4), J109.5 (Pin_5), J111.4 (Pin_4)
- net 5V: no longer names the net of J101.1 (Pin_1)
- new net: D102.1 (K), Q106.1 (D)
- new net: Q106.2 (G), R108.1, R109.1
- new net: Q107.2 (G), R111.1, R112.1
- new net: D104.2 (A), R116.2
- new net: D101.2 (A), R103.2
- new net: Q101.2 (G), R101.1, R102.1
- new net: D104.1 (K), Q108.1 (D)
- new net: D102.2 (A), R110.2
- new net: D103.1 (K), Q107.1 (D)
- new net: D103.2 (A), R113.2
- new net: D101.1 (K), Q101.1 (D)
- new net: Q108.2 (G), R114.1, R115.1
- new net 3V3_REGULATED: C101.1, C102.1, C103.1, C104.1, C105.1, C106.1, C107.1, C108.1, J107.5 (Pin_5), Q102.1 (C), Q103.1 (C), Q104.1 (C), Q105.1 (C), R103.1, R110.1, R113.1, R116.1
- new net IR_EMITTER_1: R101.2
- new net IR_EMITTER_2: R108.2
- new net IR_EMITTER_3: R111.2
- new net IR_EMITTER_4: R114.2
- new net IR_RECEIVER_1: Q102.2 (E), R104.1
- new net IR_RECEIVER_2: Q103.2 (E), R105.1
- new net IR_RECEIVER_3: Q104.2 (E), R106.1
- new net IR_RECEIVER_4: Q105.2 (E), R107.1
- new net MOTOR1_M1: J105.5 (Pin_5)
- new net MOTOR1_M2: J105.6 (Pin_6)
- new net MOTOR1_OUTA: J105.3 (Pin_3)
- new net MOTOR1_OUTB: J105.2 (Pin_2)
- new net MOTOR2_M1: J111.5 (Pin_5)
- new net MOTOR2_M2: J111.6 (Pin_6)
- new net MOTOR2_OUTA: J111.3 (Pin_3)
- new net MOTOR2_OUTB: J111.2 (Pin_2)
- new net RPI_5V: J107.3 (Pin_3)
Other:
- note added: "2x3.7 = 7.4 V Raw battery voltage --> L298N VIN Pin header connection"
- note added: "2x3.7 V Adafruit LiPoly batteries JST Connection"
- note added: "IR Receivers"
- note added: "IR Transmitters"
- note added: "NOTE: Each emitter rated for ~100 mA Eeach receiver rated for ~50 mA RPI 5V --> Step down to 3v3 using regulator --> power each receiver and transmitter from regulator output"
- note added: "Operating Current Draw ~ 40 mA 4 x 40 mA = 160 mA (receivers)"
- note added: "Operating current draw ~ 50 mA (max) 4 x 50 mA = 200 mA"
- note added: "Pololu 3V3 Regulator"
- note added: "Pololu 5V Regulator"
- note added: "Raspberry Pi 5V -> Regulator -> 3V3 for IR emitter/receiver"
- note added: "Raw Battery Voltage 7.4-8.4 V -> Regulator -> 5V for teensy input"
- note added: "Supposedly the Raspberry pi 4B 5V pin can output about 550 mA. Should be enough to power IR emitters and transmitters."
- note added: "VCC can be 2-18 V. Use 5V regulated as VCC MOTOR#_M1, MOTOR#_M2 connect to Motor Driver MOTOR#_OUTA, MOTOR#_OUTB is data sent to Teensy (Or send to Raspberry pi???)"
- note removed: "3x3.7 = 11.1 V Raw battery voltage --> L298N VIN L298 Onboard V regulator 5 V output --> Teensy 5V Pin header connection"
- note removed: "3x3.7 V Adafruit LiPoly batteries JST Connection"
- note removed: "IR Transmitters and Receivers"
- moved on the sheet: J101, J102, J103, J104, J106, U101

Commit message: general board layout established v1
Parts:
- removed J107, J109: Conn_01x05, Connector_PinHeader_2.54mm:PinHeader_1x05_P2.54mm_Vertical, symbol Connector_Generic:Conn_01x05
- removed J108, J110: Conn_01x01, Connector_PinHeader_2.54mm:PinHeader_1x01_P2.54mm_Vertical, symbol Connector_Generic:Conn_01x01
- added H101, H102, H103, H104, H105, H106, H107, H108: MountingHole_Pad, MountingHole:MountingHole_2.2mm_M2_DIN965_Pad, symbol Mechanical:MountingHole_Pad
- added H109, H110, H111, H112: MountingHole_Pad, MountingHole:MountingHole_3.2mm_M3_DIN965_Pad, symbol Mechanical:MountingHole_Pad
- added U102, U103: ~, Regulator_Pololu_D24V22FX:D24V22FX, symbol Regulator_Pololu_D24V22FX:D24V22FX
Connections:
- net 3V3_REGULATED: now also U102.5 (VOUT)
- net 5V_REGULATED: now also U103.5 (VOUT)
- net GND: now also H101.1, H102.1, H103.1, H104.1, H105.1, H106.1, H107.1, H108.1, H109.1, H110.1, H111.1, H112.1, U102.4 (GND), U102.6 (GND), U103.4 (GND), U103.6 (GND)
- net RPI_5V: now also U102.3 (VIN)
- net VBAT: now also U103.3 (VIN)
- no-connect marks 0 -> 4

Commit message: first iteration of pin assignments and routing done
Parts:
- removed H101, H102: MountingHole_Pad, MountingHole:MountingHole_2.2mm_M2_DIN965_Pad, symbol Mechanical:MountingHole_Pad
- removed J103: Conn_02x20_Odd_Even, Connector_PinHeader_2.54mm:PinHeader_2x20_P2.54mm_Vertical, symbol Connector_Generic:Conn_02x20_Odd_Even
- removed U101: Teensy4.1, MCU_TEENSY_Footprint:MODULE_DEV-16771, symbol MCU_TEENSY:Teensy4.1
- removed U103: ~, Regulator_Pololu_D24V22FX:D24V22FX, symbol Regulator_Pololu_D24V22FX:D24V22FX
- added C109: 0.1 uF, Capacitor_SMD:C_0805_2012Metric, symbol Device:C
- added C110, C111: 4.7uF, Capacitor_SMD:C_0805_2012Metric, symbol Device:C
- added C112: 10uF, Capacitor_SMD:C_0805_2012Metric, symbol Device:C
- added J103: Conn_01x10, Connector_PinHeader_2.54mm:PinHeader_1x10_P2.54mm_Vertical, symbol Connector_Generic:Conn_01x10
- added U103: L293D, Package_DIP:DIP-16_W7.62mm, symbol Driver_Motor:L293D
- added U104: Teensy4.1_bare, MCU_TEENSY_Footprint:Teensy41_bare_pins, symbol MCU_TEENSY:Teensy4.1_bare
- added U105: MCP3004, Package_DIP:DIP-14_W7.62mm, symbol Analog_ADC:MCP3004
Connections:
- net 5V_REGULATED is gone; now on net 3V3_REGULATED: J105.4 (Pin_4), J111.4 (Pin_4)
- net RPI_5V is gone; now on net VBAT: U102.3 (VIN)
- net 3V3_REGULATED: now also U103.1 (EN1,2), U103.9 (EN3,4)
- net GND: now also C109.1, C110.1, J103.4 (Pin_4), U104.1 (GND), U104.47 (GND), U105.12 (AGND), U105.7 (DGND)
- net IR_EMITTER_1: now also J103.1 (Pin_1)
- net IR_EMITTER_2: now also J103.2 (Pin_2)
- net IR_EMITTER_3: now also J103.9 (Pin_9)
- net IR_EMITTER_4: now also J103.10 (Pin_10)
- net IR_RECEIVER_1: now also U105.1 (CH0)
- net IR_RECEIVER_2: now also U105.2 (CH1)
- net IR_RECEIVER_3: now also U105.3 (CH2)
- net IR_RECEIVER_4: now also U105.4 (CH3)
- net VBAT: now also C109.2, C110.2, C111.1, C112.2, U103.16 (VCC1), U103.8 (VCC2)
- net MOTOR1_M1 renamed ML_2
- net ML_2: now also U103.3 (1Y)
- net MOTOR1_M2 renamed ML_1
- net ML_1: now also U103.6 (2Y)
- net MOTOR1_OUTA renamed ML_OUTA
- net ML_OUTA: now also U104.6 (4_BCLK2)
- net MOTOR1_OUTB renamed ML_OUTB
- net ML_OUTB: now also U104.7 (5_IN2)
- net MOTOR2_M1 renamed MR_2
- net MR_2: now also U103.11 (3Y)
- net MOTOR2_M2 renamed MR_1
- net MR_1: now also U103.14 (4Y)
- net MOTOR2_OUTA renamed MR_OUTA
- net MR_OUTA: now also U104.3 (1_TX1_CTX2_MISO1)
- net MOTOR2_OUTB renamed MR_OUTB
- net MR_OUTB: now also U104.4 (2_OUT2)
- new net MGND: C111.2, C112.1, U103.12 (GND), U103.13 (GND), U103.4 (GND), U103.5 (GND)
- new net ML_IN_1: U103.7 (2A), U104.41 (19_A5_SCL)
- new net ML_IN_2: U103.2 (1A), U104.40 (18_A4_SDA)
- new net MR_IN_1: U103.15 (4A), U104.45 (23_A9_CRX1_MCLK1)
- new net MR_IN_2: U103.10 (3A), U104.44 (22_A8_CTX1)
- new net RPI_3V3: J103.3 (Pin_3), U105.13 (Vref), U105.14 (Vdd)
- new net RPI_CLK: J103.5 (Pin_5), U105.11 (CLK)
- new net RPI_CS: J103.8 (Pin_8), U105.8 (~{CS}/SHDN)
- new net RPI_MISO: J103.6 (Pin_6), U105.10 (Dout)
- new net RPI_MOSI: J103.7 (Pin_7), U105.9 (Din)
- new net TEENSY_3V3: U104.15 (3V3), U104.46 (3V3)
- no-connect marks 4 -> 3
Other:
- note added: "Battery -> Regulator -> 3V3 for IR emitter/receiver, 3V3 for encoders Rated for 2.6A."
- note added: "IR Transmitter signal from raspberry pi SPI communication with ADC Connect to GPIO on RPI with jumper cables"
- note added: "Link to cables (female to male jumper"
- note added: "Link to female socket"
- note added: "NOTE: TEENSY, RASPBERRY PI, ADC, MOTOR DRIVER MUST ALL HAVE COMMON LOGIC GROUND (Motor driver will have seperate motor ground too)"
- note added: "Raspberry Pi Connection"
- note added: "VCC can be 2-18 V. Use 3V regulated as VCC ML_1, ML_2, MR_1, MR_2 are left and right Motor Driver outputs (inputs to motor) ML_OUTA, ML_OUTB, MR_OUTA, MR_OUTB are left and riht motor encoder data sent to Teensy (Or send to Raspberry pi???)"
- note removed: "Pololu 5V Regulator"
- note removed: "Raspberry Pi 5V -> Regulator -> 3V3 for IR emitter/receiver"
- note removed: "Raspberry Pi GPIO"
- note removed: "Raw Battery Voltage 7.4-8.4 V -> Regulator -> 5V for teensy input"
- note removed: "Receive data from IR Receiver"
- note removed: "Send data to IR Transmitter"
- note removed: "Send motor control data to Teensy"
- note removed: "TODO: pin assignments for Raspberry Pi"
- note removed: "VCC can be 2-18 V. Use 5V regulated as VCC MOTOR#_M1, MOTOR#_M2 connect to Motor Driver MOTOR#_OUTA, MOTOR#_OUTB is data sent to Teensy (Or send to Raspberry pi???)"
- moved on the sheet: J101, J102, U102

Commit message: cleaned up schematic
Parts:
- removed H109, H110, H111, H112: MountingHole_Pad, MountingHole:MountingHole_3.2mm_M3_DIN965_Pad, symbol Mechanical:MountingHole_Pad
- removed J101: Conn_01x03, Connector_PinHeader_2.54mm:PinHeader_1x03_P2.54mm_Vertical, symbol Connector_Generic:Conn_01x03
- removed J102: Conn_01x06, Connector_PinHeader_2.54mm:PinHeader_1x06_P2.54mm_Vertical, symbol Connector_Generic:Conn_01x06
Other:
- note added: "3V3 Regulator Mounting Hole"
- note added: "ADC"
- note added: "Converts Analog IR Receiver outputs into Digital signals for Raspberry Pi to read. Raspberry Pi doesnt have any Analog pins. Connect ADC output to Raspberry Pi gpio breakout"
- note added: "IR Transmitter signal from raspberry pi SPI communication with ADC Connect to GPIO on RPi with jumper cables"
- note added: "Link to UCLA IR circuit (copied from them)"
- note added: "Link to UCLA Motor Driver circuit (copied from them)"
- note added: "Motor Driver"
- note added: "Raspberry Pi Mounting Hole"
- note added: "Receives Power from USB connection with Raspberry Pi Receive motor control data from Raspberry Pi over USB (serial) Send PWM signal to Motor Driver Receive motor encoder data"
- note added: "Take PWM from teensy and output to Motors"
- note added: "VCC can be 2-18 V. Use 3V3 regulated as VCC ML_1, ML_2, MR_1, MR_2 are left and right Motor Driver outputs (inputs to motor) ML_OUTA, ML_OUTB, MR_OUTA, MR_OUTB are left and riht motor encoder data sent to Teensy (Or send to Raspberry pi???)"
- note removed: "2x3.7 = 7.4 V Raw battery voltage --> L298N VIN Pin header connection"
- note removed: "IR Transmitter signal from raspberry pi SPI communication with ADC Connect to GPIO on RPI with jumper cables"
- note removed: "L298N Motor Driver Motor Control"
- note removed: "L298N Motor Driver Power"
- note removed: "Receives Power from L298N 5 V output OR USB Receive motor control data from Raspberry Pi Send PWM signal to L298N"
- note removed: "Supposedly the Raspberry pi 4B 5V pin can output about 550 mA. Should be enough to power IR emitters and transmitters."
- note removed: "TODO: pin assignments for Teensy"
- note removed: "VCC can be 2-18 V. Use 3V regulated as VCC ML_1, ML_2, MR_1, MR_2 are left and right Motor Driver outputs (inputs to motor) ML_OUTA, ML_OUTB, MR_OUTA, MR_OUTB are left and riht motor encoder data sent to Teensy (Or send to Raspberry pi???)"
- moved on the sheet: C109, C110, C111, C112, H103, H104, H105, H106, H107, H108, J103, J104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

Commit message: updated pcb
Parts:
- added J102: Conn_02x02_Counter_Clockwise, Connector_PinHeader_2.54mm:PinHeader_2x02_P2.54mm_Vertical, symbol Connector_Generic:Conn_02x02_Counter_Clockwise
- added J108: Conn_01x04, Connector_PinHeader_2.54mm:PinHeader_1x04_P2.54mm_Vertical, symbol Connector_Generic:Conn_01x04
- added SW101: SW_SPST, Connector_PinHeader_2.54mm:PinHeader_1x02_P2.54mm_Vertical, symbol Switch:SW_SPST
- R103: value 50 Ohm -> 51Ohm
- R110, R113: value 50 Ohm -> 51 Ohm
Connections:
- net 3V3_REGULATED: now also J108.1 (Pin_1)
- net GND: now also J108.3 (Pin_3)
- net MGND: now also J108.4 (Pin_4)
- net ML_OUTA: now also J102.3 (Pin_3)
- net ML_OUTB: now also J102.1 (Pin_1)
- net MR_OUTA: now also J102.4 (Pin_4)
- net MR_OUTB: now also J102.2 (Pin_2)
- net VBAT: now also J108.2 (Pin_2), SW101.2 (B); no longer J104.1 (Pin_1)
- net TEENSY_3V3: no longer names the net of U104.15 (3V3)
- net TEENSY_3V3: no longer U104.46 (3V3)
- new net: J104.1 (Pin_1), SW101.1 (A)
Other:
- note added: "Connection to Raspberry Pi"
- note added: "Debug Pins"
- moved on the sheet: J104, J106

Commit message: added mounting holes
Other:
- moved on the sheet: J108
Changed lines of the file:
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@@
 	(wire
 		(pts
-			(xy 381 60.96) (xy 391.16 60.96)
+			(xy 383.54 35.56) (xy 393.7 35.56)
 		)
 		(stroke
@@
 	(hierarchical_label "3V3_REGULATED"
 		(shape input)
-		(at 391.16 55.88 180)
+		(at 393.7 30.48 180)
 		(fields_autoplaced yes)
 		(effects
@@
 	(hierarchical_label "VBAT"
 		(shape input)
-		(at 391.16 58.42 180)
+		(at 393.7 33.02 180)
 		(fields_autoplaced yes)
 		(effects
@@
 	(hierarchical_label "MGND"
 		(shape input)
-		(at 391.16 63.5 180)
+		(at 393.7 38.1 180)
 		(fields_autoplaced yes)
 		(effects
@@
 	(symbol
 		(lib_id "power:GND")
-		(at 381 60.96 0)
+		(at 383.54 35.56 0)
 		(unit 1)
 		(exclude_from_sim no)
@@
 		(fields_autoplaced yes)
 		(property "Reference" "#PWR0101"
-			(at 381 67.31 0)
+			(at 383.54 41.91 0)
 			(effects
 				(font
@@
 		)
 		(property "Value" "GND"
-			(at 381 66.04 0)
+			(at 383.54 40.64 0)
 			(effects
 				(font
@@
 		)
 		(property "Footprint" ""
-			(at 381 60.96 0)
+			(at 383.54 35.56 0)
 			(effects
 				(font
@@
 		)
 		(property "Datasheet" ""
-			(at 381 60.96 0)
+			(at 383.54 35.56 0)
 			(effects
 				(font
@@
 		)
 		(property "Description" "Power symbol creates a global label with name \"GND\" , ground"
-			(at 381 60.96 0)
+			(at 383.54 35.56 0)
 			(effects
 				(font
@@
 	(symbol
 		(lib_id "Connector_Generic:Conn_01x04")
-		(at 396.24 58.42 0)
+		(at 398.78 33.02 0)
 		(unit 1)
 		(exclude_from_sim no)
@@
 		(on_board yes)
 		(dnp no)
-		(fields_autoplaced yes)
 		(property "Reference" "J108"
-			(at 398.78 58.4199 0)
+			(at 401.32 33.0199 0)
 			(effects
 				(font
@@
 		)
 		(property "Value" "Conn_01x04"
-			(at 398.78 60.9599 0)
+			(at 401.32 35.5599 0)
 			(effects
 				(font
@@
 		)
 		(property "Footprint" "Connector_PinHeader_2.54mm:PinHeader_1x04_P2.54mm_Vertical"
-			(at 396.24 58.42 0)
+			(at 398.78 33.02 0)
 			(effects
 				(font
@@
 		)
 		(property "Datasheet" "~"
-			(at 396.24 58.42 0)
+			(at 398.78 33.02 0)
 			(effects
 				(font
@@
 		)
 		(property "Description" "Generic connector, single row, 01x04, script generated (kicad-library-utils/schlib/autogen/connector/)"
-			(at 396.24 58.42 0)
+			(at 398.78 33.02 0)
 			(effects
 				(font
